File: PCB/QdecLogic.sch (EAGLE design)
At the start: 0 parts

Commit message: schematic layout
Parts:
- added J1, J2, J3, J4: (no value), SparkFun-Connectors:M02PTH
- added U$1: D-TYPE_FLIPFLOP, AmandaEagleLibrary:D-TYPE_FLIPFLOP
- added U$2: AND_GATE_2CH, AmandaEagleLibrary:AND_GATE_2CH
Connections:
- new net A: J1.2, U$1.D, U$2.1B, U$2.2B
- new net B: J1.1, U$1.CLK
- new net DEC: J2.1, U$2.2OUT
- new net GND: U$1.GND, U$2.GND
- new net INCR: J2.2, U$2.1OUT
- new net N$5: U$1.Q, U$2.1A
- new net N$6: U$1.!Q, U$2.2A
- new net VCC: U$1.!CLR, U$1.!PR, U$1.VCC, U$2.VCC
