File: PCB/QdecLogic.sch (EAGLE design)
At the start: 6 parts

Commit message: pngs
Parts:
- added J5, J6: (no value), SparkFun-Connectors:M02PTH
- added R1, R2: 0, fab:RES-US1206FAB
Connections:
- removed net N$5: U$1.Q, U$2.1A
- new net DIR: J4.1, U$1.Q, U$2.1A
- net GND: now also J3.1
- net VCC: now also J3.2
Other:
- moved on the sheet: J4
Changed lines of the file:
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@@
 <part name="J3" library="SparkFun-Connectors" deviceset="M02" device="PTH"/>
 <part name="J4" library="SparkFun-Connectors" deviceset="M02" device="PTH"/>
+<part name="R1" library="fab" deviceset="RES-US" device="1206FAB" value="0"/>
+<part name="R2" library="fab" deviceset="RES-US" device="1206FAB" value="0"/>
+<part name="J5" library="SparkFun-Connectors" deviceset="M02" device="PTH"/>
+<part name="J6" library="SparkFun-Connectors" deviceset="M02" device="PTH"/>
 </parts>
 <sheets>
@@
 <instance part="GND1" gate="1" x="66.04" y="45.72"/>
 <instance part="J3" gate="G$1" x="53.34" y="106.68"/>
-<instance part="J4" gate="G$1" x="66.04" y="106.68"/>
+<instance part="J4" gate="G$1" x="81.28" y="106.68"/>
+<instance part="R1" gate="G$1" x="30.48" y="114.3"/>
+<instance part="R2" gate="G$1" x="30.48" y="106.68"/>
+<instance part="J5" gate="G$1" x="104.14" y="106.68"/>
+<instance part="J6" gate="G$1" x="116.84" y="106.68"/>
 </instances>
 <busses>
@@
 </segment>
 </net>
-<net name="N$5" class="0">
-<segment>
-<pinref part="U$1" gate="G$1" pin="Q"/>
-<pinref part="U$2" gate="G$1" pin="1A"/>
-<wire x1="58.42" y1="76.2" x2="81.28" y2="76.2" width="0.1524" layer="91"/>
-</segment>
-</net>
 <net name="N$6" class="0">
 <segment>
@@
 <junction x="27.94" y="66.04"/>
 </segment>
+<segment>
+<pinref part="J3" gate="G$1" pin="2"/>
+<wire x1="60.96" y1="109.22" x2="66.04" y2="109.22" width="0.1524" layer="91"/>
+<label x="60.96" y="109.22" size="1.778" layer="95"/>
+</segment>
 </net>
 <net name="GND" class="0">
@@
 <junction x="66.04" y="55.88"/>
 </segment>
+<segment>
+<pinref part="J3" gate="G$1" pin="1"/>
+<wire x1="60.96" y1="106.68" x2="66.04" y2="106.68" width="0.1524" layer="91"/>
+<label x="60.96" y="106.68" size="1.778" layer="95"/>
+</segment>
 </net>
+<net name="DIR" class="0">
+<segment>
+<pinref part="J4" gate="G$1" pin="1"/>
+<wire x1="88.9" y1="106.68" x2="96.52" y2="106.68" width="0.1524" layer="91"/>
+<label x="91.44" y="106.68" size="1.778" layer="95"/>
+</segment>
+<segment>
+<pinref part="U$1" gate="G$1" pin="Q"/>
+<pinref part="U$2" gate="G$1" pin="1A"/>
+<wire x1="58.42" y1="76.2" x2="81.28" y2="76.2" width="0.1524" layer="91"/>
+<label x="66.04" y="76.2" size="1.778" layer="95"/>
+</segment>
+</net>

Commit message: fixed pcb layout
Connections:
- net A: now also U$1.CLK; no longer U$1.D
- net B: now also U$1.D; no longer U$1.CLK
Changed lines of the file:
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@@
-</segment>
-<segment>
-<pinref part="U$1" gate="G$1" pin="D"/>
-<wire x1="27.94" y1="76.2" x2="17.78" y2="76.2" width="0.1524" layer="91"/>
-<label x="20.32" y="76.2" size="1.778" layer="95"/>
 </segment>
 <segment>
@@
 <label x="73.66" y="66.04" size="1.778" layer="95"/>
 </segment>
+<segment>
+<pinref part="U$1" gate="G$1" pin="CLK"/>
+<wire x1="27.94" y1="71.12" x2="17.78" y2="71.12" width="0.1524" layer="91"/>
+<label x="20.32" y="71.12" size="1.778" layer="95"/>
+</segment>
 </net>
 <net name="B" class="0">
@@
 </segment>
 <segment>
-<pinref part="U$1" gate="G$1" pin="CLK"/>
-<wire x1="27.94" y1="71.12" x2="17.78" y2="71.12" width="0.1524" layer="91"/>
-<label x="20.32" y="71.12" size="1.778" layer="95"/>
+<pinref part="U$1" gate="G$1" pin="D"/>
+<wire x1="27.94" y1="76.2" x2="17.78" y2="76.2" width="0.1524" layer="91"/>
+<label x="20.32" y="76.2" size="1.778" layer="95"/>
 </segment>
 </net>

Commit message: v2
Parts:
- removed J1, J2, J3, J4, J5, J6: (no value), SparkFun-Connectors:M02PTH
- removed R1, R2: 0, fab:RES-US1206FAB
- added J10, J9: (no value), SparkFun-Connectors:M01PTH_NO_SILK_YES_STOP
- added J7, J8: (no value), SparkFun-Connectors:M05NO_SILK
- U$1: value D-TYPE_FLIPFLOP -> AND_GATE_4CH; device AmandaEagleLibrary:D-TYPE_FLIPFLOP -> AmandaEagleLibrary:AND_GATE_4CH
- U$2: value AND_GATE_2CH -> FLIPFLOP_D-TYPE_2CH; device AmandaEagleLibrary:AND_GATE_2CH -> AmandaEagleLibrary:FLIPFLOP_D-TYPE_2CH
Connections:
- removed net A: J1.2, U$1.CLK, U$2.1B, U$2.2B
- removed net B: J1.1, U$1.D
- removed net DEC: J2.1, U$2.2OUT
- removed net DIR: J4.1, U$1.Q, U$2.1A
- removed net INCR: J2.2, U$2.1OUT
- new net A1: J7.5, U$2.D1
- new net A2: J8.5, U$2.D2
- new net B1: J7.4, U$1.IN1B, U$1.IN2B, U$2.CP1
- new net B2: J8.4, U$1.IN3B, U$1.IN4B, U$2.CP2
- new net DIR1: J7.3, U$1.IN1A, U$2.Q1
- new net DIR2: J8.3, U$1.IN3A, U$2.Q2
- new net FWD1: J7.2, U$1.OUT1
- new net FWD2: J8.2, U$1.OUT3
- new net N$8: U$1.IN4A, U$2.!Q2
- new net REV1: J7.1, U$1.OUT2
- new net REV2: J8.1, U$1.OUT4
- net GND: now also J9.1; no longer J3.1
- net N$6: now also U$1.IN2A, U$2.!Q1; no longer U$1.!Q, U$2.2A
- net VCC: now also J10.1, U$2.!RD1, U$2.!RD2, U$2.!SD1, U$2.!SD2; no longer J3.2, U$1.!CLR, U$1.!PR
