File: PCB/QdecLogic.brd (EAGLE design)
At the start: 160 x 100 mm, 6 parts

Commit message: pngs
Parts:
- added J5, J6: (no value), SparkFun-Connectors:1X02
- added R1, R2: 0, fab:R1206FAB
- moved J3 13.7 mm to (34.3, 10.2)
- moved J4 12.7 mm to (34.3, 22.9)
- moved J2 5.08 mm to (29.2, 22.9)
- moved U$2 3.35 mm to (31.0, 18.6)
- moved U$1 2.54 mm to (34.3, 15.2)
Connections:
- removed net N$5: U$1.P$5, U$2.P$1
- new net DIR: J4.1, U$1.P$5, U$2.P$1
- net GND: now also J3.1
- net VCC: now also J3.2
Routing:
- net A: track 0.00 -> 26.4 mm
- net GND: track 0.00 -> 21.0 mm
- net DEC: track 0.00 -> 15.8 mm
- net N$6: track 0.00 -> 15.2 mm
- net VCC: track 0.00 -> 12.9 mm
- net DIR: track 0.00 -> 9.40 mm
- net B: track 0.00 -> 7.36 mm
- net INCR: track 0.00 -> 5.01 mm

Commit message: fixed pcb layout
Parts:
- moved J1 2.54 mm to (31.8, 10.2), turned to 180 degrees
Connections:
- net A: now also U$1.P$1; no longer U$1.P$2
- net B: now also U$1.P$2; no longer U$1.P$1
Routing:
- net B: track 7.36 -> 4.75 mm
- net A: track 26.4 -> 25.6 mm

Commit message: v2
Parts:
- removed J1, J2, J3, J4, J5, J6: (no value), SparkFun-Connectors:1X02
- removed R1, R2: 0, fab:R1206FAB
- added J10, J9: (no value), SparkFun-Connectors:1X01_NO_SILK
- added J7, J8: (no value), SparkFun-Connectors:1X05_NO_SILK
- U$1: value D-TYPE_FLIPFLOP -> AND_GATE_4CH; device AmandaEagleLibrary:US8_8-LEAD -> AmandaEagleLibrary:14-SOIC
- U$2: value AND_GATE_2CH -> FLIPFLOP_D-TYPE_2CH; device AmandaEagleLibrary:US8_8-LEAD -> AmandaEagleLibrary:14-SOIC
- moved U$2 12.9 mm to (43.2, 22.9), turned to 0 degrees
- moved U$1 9.67 mm to (43.2, 11.4)
Connections:
- removed net A: J1.2, U$1.P$1, U$2.P$2, U$2.P$6
- removed net B: J1.1, U$1.P$2
- removed net DEC: J2.1, U$2.P$7
- removed net DIR: J4.1, U$1.P$5, U$2.P$1
- removed net INCR: J2.2, U$2.P$3
- new net A1: J7.5, U$2.2
- new net A2: J8.5, U$2.12
- new net B1: J7.4, U$1.2, U$1.5, U$2.3
- new net B2: J8.4, U$1.10, U$1.13, U$2.11
- new net DIR1: J7.3, U$1.1, U$2.5
- new net DIR2: J8.3, U$1.9, U$2.9
- new net FWD1: J7.2, U$1.3
- new net FWD2: J8.2, U$1.8
- new net N$8: U$1.12, U$2.8
- new net REV1: J7.1, U$1.6
- new net REV2: J8.1, U$1.11
- net GND: now also J9.1, U$1.7, U$2.7; no longer J3.1, U$1.P$4, U$2.P$4
- net N$6: now also U$1.4, U$2.6; no longer U$1.P$3, U$2.P$5
- net VCC: now also J10.1, U$1.14, U$2.1, U$2.10, U$2.13, U$2.14, U$2.4; no longer J3.2, U$1.P$6, U$1.P$7, U$1.P$8, U$2.P$8
Routing:
- net B2: track 0.00 -> 28.7 mm, vias 0 -> 2
- net B1: track 0.00 -> 26.0 mm, vias 0 -> 2
- net A: track 25.6 -> 0.00 mm
- net VCC: track 12.9 -> 35.1 mm
- net DIR2: track 0.00 -> 20.6 mm
- net DEC: track 15.8 -> 0.00 mm
- net DIR1: track 0.00 -> 13.6 mm
- net FWD2: track 0.00 -> 13.2 mm
- net N$8: track 0.00 -> 11.3 mm
- net REV2: track 0.00 -> 11.0 mm, vias 0 -> 2
- net DIR: track 9.40 -> 0.00 mm
- net REV1: track 0.00 -> 9.11 mm
- net A2: track 0.00 -> 7.57 mm
- net FWD1: track 0.00 -> 7.08 mm
- net A1: track 0.00 -> 7.08 mm
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- added copper zone on layer 16, net GND
