File: PCB/Tiny45Logic.brd (EAGLE design)
At the start: 160 x 100 mm, 6 parts

Commit message: attiny45
Parts:
- removed J10, J9: (no value), SparkFun-Connectors:1X01_NO_SILK
- removed J7, J8: (no value), SparkFun-Connectors:1X05_NO_SILK
- removed U$1: AND_GATE_4CH, AmandaEagleLibrary:14-SOIC
- removed U$2: FLIPFLOP_D-TYPE_2CH, AmandaEagleLibrary:14-SOIC
- added J1, J2: (no value), SparkFun-Connectors:1X02
- added J3, J4: (no value), SparkFun-Connectors:1X01
- added JP1: (no value), fab:2X03SMD
- added R1: 1K, fab:R1206
- added U1: Tiny45-20-SMT, SparkFun-DigitalIC:SO08-EIAJ
Connections:
- removed net A1: J7.5, U$2.2
- removed net A2: J8.5, U$2.12
- removed net B1: J7.4, U$1.2, U$1.5, U$2.3
- removed net B2: J8.4, U$1.10, U$1.13, U$2.11
- removed net DIR1: J7.3, U$1.1, U$2.5
- removed net DIR2: J8.3, U$1.9, U$2.9
- removed net FWD1: J7.2, U$1.3
- removed net FWD2: J8.2, U$1.8
- removed net N$6: U$1.4, U$2.6
- removed net N$8: U$1.12, U$2.8
- removed net REV1: J7.1, U$1.6
- removed net REV2: J8.1, U$1.11
- removed net VCC: J10.1, U$1.14, U$2.1, U$2.10, U$2.13, U$2.14, U$2.4
- new net 3.3V: J3.1, JP1.2, R1.2, U1.8
- new net FWD: J2.1, U1.2
- new net MISO: J1.2, JP1.1, U1.6
- new net MOSI: J1.1, JP1.4, U1.5
- new net REV: J2.2, U1.3
- new net RST: JP1.5, R1.1, U1.1
- new net SCK: JP1.3, U1.7
- net GND: now also J4.1, JP1.6, U1.4; no longer J9.1, U$1.7, U$2.7
Routing:
- net VCC: track 35.1 -> 0.00 mm
- net RST: track 0.00 -> 31.2 mm
- net B2: track 28.7 -> 0.00 mm, vias 2 -> 0
- net B1: track 26.0 -> 0.00 mm, vias 2 -> 0
- net DIR2: track 20.6 -> 0.00 mm
- net MOSI: track 0.00 -> 18.4 mm
- net GND: track 15.2 -> 0.00 mm, vias 2 -> 0
- net N$6: track 13.9 -> 0.00 mm, vias 2 -> 0
- net DIR1: track 13.6 -> 0.00 mm
- net FWD2: track 13.2 -> 0.00 mm
- net N$8: track 11.3 -> 0.00 mm
- net REV2: track 11.0 -> 0.00 mm, vias 2 -> 0
- net 3.3V: track 0.00 -> 9.77 mm
- net SCK: track 0.00 -> 9.18 mm
- net REV1: track 9.11 -> 0.00 mm
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- added copper zone on layer 1, net GND
- removed copper zone on layer 16, net GND

Commit message: eod
Connections:
- net MISO renamed MISO/B
- net MOSI renamed MOSI/A
Changed lines of the file:
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@@
 </elements>
 <signals>
-<signal name="MOSI">
+<signal name="MOSI/A">
 <contactref element="U1" pad="5"/>
 <contactref element="JP1" pad="4"/>
@@
 <wire x1="11.43" y1="26.035" x2="11.1125" y2="26.3525" width="0.6096" layer="1"/>
 </signal>
-<signal name="MISO">
+<signal name="MISO/B">
 <contactref element="U1" pad="6"/>
 <contactref element="JP1" pad="1"/>

Commit message: caps
Parts:
- added C1: 0.1uF, fab:C1206FAB
- added C2: 10uF, fab:C1206FAB
- moved J4 0.63 mm to (11.4, 38.7)
- moved J2 0.63 mm to (16.5, 38.7)
Connections:
- net 3.3V: now also C1.1, C2.1
- net GND: now also C1.2, C2.2
Routing:
- net 3.3V: track 9.77 -> 14.5 mm
- net GND: track 0.00 -> 2.54 mm
